Commit message: Add realsense camera

File: src/example_robot_description/urdf/accessories.urdf.xacro (robot description, xacro)
@@ -58,4 +58,10 @@
       <child link="$(optenv JACKAL_FLEA3_MOUNT front)_camera" />
     </joint>
+  </xacro:if>
+  <xacro:if value="$(optenv JACKAL_REALSENSE 0)">
+    <xacro:include filename="$(find example_robot_description)/urdf/realsense_d435.urdf.xacro" />
+    <xacro:realsense_d435 parent="front_mount" name="realsense">
+      <origin xyz="0.1 0 0" rpy="0 0 0" />
+    </xacro:realsense_d435>
   </xacro:if>
   <xacro:include filename="$(find example_robot_description)/urdf/accessories/stereo_camera_mount.urdf.xacro" />
